File: schematics/schematics.kicad_sch (KiCad schematic)
At the start: 36 parts, among them U1 N2N, U2 V2B, U3 D24, U5 D24

Commit message: New speculative cells
Parts:
- added A18, A96, B12, C1, C2, C3, C69, D11, D61, E114, E115, E116, F6, G32, G33, G34, G39, G7, G8, H51, H67, I47, K57, K61, K62, K63, K64, K65, K66, K82, K83, K94, M53, M54, M55, M56, Q105, Q11, Q120, Q28, Q91, Q92, U10, U12, U13, U14, U15, U16, U17, U44, U45, U47, U61, U9: N2N, symbol ga_fujitsu_av:N2N
- added A19, A36, A39, B9, C10, D2, D62, D63, D64, D7, D8, E55, E56, F3, G11, G60, I27, I29, I46, K101, K102, K103, K56, K67, K96, M57, O27, Q10, Q16, Q2, Q3, Q6, T32, U11, U18, U19, U23, U24, U46: V2B, symbol ga_fujitsu_av:V2B
- added A20, A4, A75, B61, B74, B87, K20, K3, K34, N61, N77, N93, O108, O61, O75, O95, P92, Q107, R107, R61, R93, S106, T17, T33, T4, U31: LT4, symbol ga_fujitsu_av:LT4
- added A3, A47, A48, F92, G2, G20, G6, G63, G64, G65, G66, H52, H55, H56, H61, H62, H63, I15, I20, I28, I45, I48, I49, I60, J56, K16, K58, M58, N15, U20, U25, U30, U48, U51, U54, U7, U8: V1N, symbol ga_fujitsu_av:V1N
- added A34, A37, A49, A51, A53, A55, A57, A59, A61, A63, A65, A67, A90, A92, A94, C61, C63, C65, C67, G4, G61, H53, H57, H59, H64, I115, I117, I119, I16, I18, I50, J57, J59, J61, J63, K18, K59, K68, K70, K72, K74, L107, L109, L111, L113, L94, L96, L98, M101, M103, M108, M110, M112, M59, N13, P61, P77, P79, P87, P89, Q61, Q69, Q71, Q73, Q88, R26, R88, R90, S119, S81, S83, S91, U21, U26, U28, U49, U52, U55: D24, symbol ga_fujitsu_av:D24
- added A40, A43: K4B, symbol ga_fujitsu_av:K4B
- added A69, K48, K52: UNKC, symbol ga_fujitsu_av:UNKC
- added A98, B100, D66, D96, F61, F94, S10: FDQ, symbol ga_fujitsu_av:FDQ
- added B1, C4, F7, G40, K87, L100, L115, L61, L67, L75, L81, L87, M114, M61, M67, M75, M81, M89, M95, P63, P69, P81, Q63, Q76, Q82, Q93, Q99, S61, S67, S73, S85, S99: FDM, symbol ga_fujitsu_av:FDM
- added B10, C11, E117, E119, F1, G35, G37, G9, O23, O25, O47, Q26, Q32, Q4, T2: N2P, symbol ga_fujitsu_av:N2P
- added B13, C13, D13, E7, F13: C43, symbol ga_fujitsu_av:C43
- added B7, D9, T30: N3N, symbol ga_fujitsu_av:N3N
- added C71, E61, G68, H1, H69, I61, J6, J66, M3, T69, U69: A4H, symbol ga_fujitsu_av:A4H
- added D3, D5, E57: N4N, symbol ga_fujitsu_av:N4N
- added D91, E2: X1B, symbol ga_fujitsu_av:X1B
- added E59, F4, N16, N18, N20, N22, N24, N32, N34, N36, N38, N40, N42, N44, O49, O51, O53, O55, O57, O59, Q7, T46: R2P, symbol ga_fujitsu_av:R2P
- added F90, I58: K1B, symbol ga_fujitsu_av:K1B
- added G12: UNKG, symbol ga_fujitsu_av:UNKG
- added G21: FDD, symbol ga_fujitsu_av:FDD
- added G3, K100, K105, K106, K107, K108, K109, K110, K78, K79, K80, K81, K95, K97, K98, K99, L20, L40, L60, Q29, Q45, Q9, R120, T61, T62, T63, T64, T65, T66, T67: R2N, symbol ga_fujitsu_av:R2N
- added G46, G50, N5, N9, O11, O28, O3, O7, P112, P116: X2B, symbol ga_fujitsu_av:X2B
- added G54, G57, N2: R2B, symbol ga_fujitsu_av:R2B
- added K111, K114, K117, K84: K2B, symbol ga_fujitsu_av:K2B
- added N109, O88, P106, R76, R82, S93, U62: U34, symbol ga_fujitsu_av:U24
- added N115: DE2, symbol ga_fujitsu_av:DE2
- added N26, O33: N8B, symbol ga_fujitsu_av:N8B
- added N46: DE3, symbol ga_fujitsu_av:DE3
- added O16: FDN, symbol ga_fujitsu_av:FDN
- added O39: FDO, symbol ga_fujitsu_av:FDO
- added P1, P10, P19, P35, P52, Q17, Q36, Q52, R17, R2, R28, R37, R52: UNKH, symbol ga_fujitsu_av:UNKH
- added P28: FD6, symbol ga_fujitsu_av:FD6
- added P44: UNKA, symbol ga_fujitsu_av:UNKA
- added P46, R11, R46: UNKD, symbol ga_fujitsu_av:UNKD
- added Q12, Q34: D23, symbol ga_fujitsu_av:D23
- added Q14, Q30: UNKB, symbol ga_fujitsu_av:UNKB
- added Q46: UNKE, symbol ga_fujitsu_av:UNKE
- added S1, S31, S34, S37, S4, S40, S43, S46, S49, S52, S55, S58, S7, T48, T51, T54: R4P, symbol ga_fujitsu_av:R4P
- added T57, U57: N4B, symbol ga_fujitsu_av:N4B

Commit message: Stuff!
Parts:
- removed A19, A36, B9, D2, D62, D63, D7, D8, E55, E56, G11, G60, I29, K101, K102, K103, K56, K67, K96, M57, O27, Q10, Q16, Q2, Q3, Q6, U19, U2, U23, U24, U46: V2B, symbol ga_fujitsu_av:V2B
- removed A20, A4, A75, B61, B74, B87, K20, K3, N61, N77, N93, O108, O61, O75, O95, P92, Q107, R107, R61, R93, S106, V78: LT4, symbol ga_fujitsu_av:LT4
- removed A3, A47, A48, F92, G2, G20, G6, G63, G64, G65, G66, H52, H55, H56, H61, H62, H63, I15, I20, I28, I45, I48, I49, I60, J56, K16, K58, M58, N15, U20, U25, U30, U48, U51, U54, U7, U8: V1N, symbol ga_fujitsu_av:V1N
- removed A34, A37, A49, A51, A53, A55, A57, A59, A61, A63, A65, A67, A90, A92, A94, C61, C63, C65, C67, G4, G61, H53, H57, H59, H64, I115, I117, I119, I16, I18, I50, J57, J59, J61, J63, K18, K59, K68, K70, K72, K74, L107, L109, L111, L113, L94, L96, L98, M101, M103, M108, M110, M112, M59, N13, P61, P77, P79, P87, P89, Q61, Q69, Q71, Q73, Q88, R26, R88, R90, S119, S81, S83, S91, U21, U26, U28, U3, U49, U5, U52, U55: D24, symbol ga_fujitsu_av:D24
- removed A69: UNKC, symbol ga_fujitsu_av:UNKC
- removed A98, B100, D66, D96, F61, F94, S10, V10: FDQ, symbol ga_fujitsu_av:FDQ
- removed B1, K87, L100, L115, L61, L67, L75, L81, L87, M114, M61, M67, M75, M81, M89, M95, P63, P69, P81, Q63, Q76, Q82, Q93, Q99, S61, S67, S73, S85, S99, V99: FDM, symbol ga_fujitsu_av:FDM
- removed B10, E117, E119, F1, G35, G37, G9, O23, O25, O47, Q26, Q32, Q4, T2: N2P, symbol ga_fujitsu_av:N2P
- removed B12, D61, E116, G7, G8, K57, K61, K62, K63, K64, K65, K66, K82, K83, K94, M53, M54, M55, M56, Q105, Q11, Q120, Q28, Q91, Q92, U1, U61, V105, V75, V98: N2N, symbol ga_fujitsu_av:N2N
- removed B7, D9, T30: N3N, symbol ga_fujitsu_av:N3N
- removed C71, E61, G68, H1, H69, I61, J6, J66, M3, T69, U69: A4H, symbol ga_fujitsu_av:A4H
- removed D13, E7: C43, symbol ga_fujitsu_av:C43
- removed D91, E2: X1B, symbol ga_fujitsu_av:X1B
- removed E57: N4N, symbol ga_fujitsu_av:N4N
- removed E59, F4, N16, N18, N20, N22, N24, N32, N34, N36, N38, N40, N42, O49, O51, O53, O55, O57, O59, Q7, T46: R2P, symbol ga_fujitsu_av:R2P
- removed F90, I58: K1B, symbol ga_fujitsu_av:K1B
- removed G21: FDD, symbol ga_fujitsu_av:FDD
- removed G3, K100, K105, K106, K107, K108, K109, K110, K78, K79, K80, K81, K95, K97, K98, K99, L20, L40, L60, Q29, Q45, Q9, R120, T61, T62, T63, T64, T65, T66, T67: R2N, symbol ga_fujitsu_av:R2N
- removed G46, G50, N5, N9, O11, O28, O3, O7, P112, P116: X2B, symbol ga_fujitsu_av:X2B
- removed G54, G57: R2B, symbol ga_fujitsu_av:R2B
- removed K111, K114, K117, K84: K2B, symbol ga_fujitsu_av:K2B
- removed N109, O88, P106, R76, R82, S93, U62, V91: U34, symbol ga_fujitsu_av:U24
- removed N115: DE2, symbol ga_fujitsu_av:DE2
- removed N26, O33: N8B, symbol ga_fujitsu_av:N8B
- removed N46: DE3, symbol ga_fujitsu_av:DE3
- removed O16: FDN, symbol ga_fujitsu_av:FDN
- removed O39: FDO, symbol ga_fujitsu_av:FDO
- removed P1, P10, P19, P35, P52, Q17, Q36, Q52, R17, R2, R28, R37, R52: UNKH, symbol ga_fujitsu_av:UNKH
- removed P28: FD6, symbol ga_fujitsu_av:FD6
- removed P44: UNKA, symbol ga_fujitsu_av:UNKA
- removed P46, R11, R46: UNKD, symbol ga_fujitsu_av:UNKD
- removed Q12, Q34: D23, symbol ga_fujitsu_av:D23
- removed Q14, Q30: UNKB, symbol ga_fujitsu_av:UNKB
- removed Q46: UNKE, symbol ga_fujitsu_av:UNKE
- removed S1, S31, S34, S37, S4, S40, S43, S46, S49, S52, S55, S58, S7, T48, T51, T54: R4P, symbol ga_fujitsu_av:R4P
- added P28: UNKF, symbol ga_fujitsu_av:UNKF
Connections:
- net at C10.1: now also C4.3 (Q)
- net at C10.2: now also C11.1
- net 9_FSYNC_IN: now reaches F13.5 (L)
- net 10_SYNC_IN: now reaches F13.6 (CK)
- net 10_SYNC_IN: now also A40.1, A43.2
- net AD_WRITE_LOW?: now reaches K34. (~{Q3})
- net AD_WRITE_LOW?: now also G12.2 (CK), K48.1, K52.1, T33. (~{Q3}), T57.5, V48. (~{Q3}), V61. (~{Q3})
- net at A39.1: now also A43.1
- net at A39.2: now also A40.2
- net at A40.3: now also N44.1
- net 45_AL7_IN: now reaches V120.1
- net at V120.2: now also U11.2, V32.2, V46.2, V6.1, V74.2, V77.2, V8.2, V9.2, V97.2
- net at V120.3: now also V31.2
- net at T57.1: now also U57.1, V107.4
- net at T57.2: now also U10.3, U18.1
- net at T57.3: now also T32.2, U57.3, V47.1
- net 68_E_IN: now reaches T57.4
- net 68_E_IN: now also G12.1 (D), U44.2, U57.4, V47.2
- net AD_LATCHED_2: now reaches K48.2
- net AD_LATCHED_2: now also U17.3
- net at E114.1: now also C2.3
- net at E114.2: now also G32.3
- net 28_RIC12_A5_OUT: now reaches E114.3
- net at I27.1: now also N44.3
- net at I27.2: now also G40.2 (CK)
- net at V2.1: now also V3.3
- net at V2.2: now also V97.3
- net 60_AL0_IN: now reaches V8.1
- net 60_AL0_IN: now also V61. (~{Q3})
- net at V8.3: now also U10.2
- net at N2.3: now also C4.2 (CK)
- net 58_AL1_IN: now reaches V9.1
- net 58_AL1_IN: now also V61. (~{Q3})
- net at V9.3: now also U9.2
- net at D5.5: now also D11.1
- net 49_AL5_OUT: now reaches V4.1
- net 49_AL5_OUT: now also V33. (~{Q3})
- net 76_AL_CT_IN: now reaches V4.2
- net 76_AL_CT_IN: now also U11.1, U12.2, U13.2, U14.2, U15.2, U45.2, V1.2, V3.2
- net at V4.3: now also U16.1
- net 53_WR_OUT: now reaches V47.3
- net at C1.3: now also H67.1
- net 56_AL2_OUT: now reaches U12.1
- net 56_AL2_OUT: now also T4. (~{Q3})
- net at U12.3: now also U17.1
- net at E115.1: now also I47.3
- net at E115.2: now also G39.1, G40.3 (Q)
- net 27_RIC12_WE_OUT: now reaches E115.3
- net 51_AL4_IN: now reaches V74.1
- net at V74.3: now also U47.2
- net 60_AL0_OUT: now reaches U15.1
- net 60_AL0_OUT: now also T4. (~{Q3})
- net at U15.3: now also U10.1
- net at C3.3: now also C69.1
- net 43_P47_IN: now reaches V113.1
- net 43_P47_IN: now also V114.1
- net 78_P46_IN: now reaches V113.2
- net 78_P46_IN: now also V114.2
- net at V113.3: now also V107.1, V110.1
- net at U57.2: now also U18.2
- net AD_WRITE_HIGH?: now reaches U57.5
- net AD_WRITE_HIGH?: now also T17. (~{Q3}), U31. (~{Q3})
- net 74_UNK_IN: now reaches C11.2
- net 74_UNK_IN: now also G12.3 (S), V6.2
- net RIC12_D_OE: now reaches C11.3
- net at D64.1: now also C4.4 (~{Q})
- net 25_RIC12_OE_OUT: now reaches D64.2
- net at I46.2: now also G39.2
- net at U9.1: now also U14.3
- net AD_LATCHED_1: now reaches U9.3
- net AD_LATCHED_1: now also K52.2
- net at V118.1: now also V114.3
- net 55_RD_OUT: now reaches V118.2
- net 55_RD_OUT: now also U44.3
- net 42_PARAM_ROMCS_OUT: now reaches V118.3
- net at U17.2: now also V32.3
- net at A18.3: now also A96.1
- net 58_AL1_OUT: now reaches U14.1
- net 58_AL1_OUT: now also T4. (~{Q3})
- net 44_P45_I4: now reaches V107.2
- net 44_P45_I4: now also V110.2
- net 46_P44_IN: now reaches V107.3
- net 46_P44_IN: now also V112.1
- net 70_RW_IN: now reaches U44.1
- net 70_RW_IN: now also T32.1
- net at F6.3: now also F7.1 (D)
- net at F3.1: now also F7.4 (~{Q})
- net at F3.2: now also G32.2, G33.2, G34.2, H51.2
- net 47_AL6_IN: now reaches V97.1
- net at G34.1: now also K34. (~{Q3})
- net at G34.3: now also C69.2
- net at G12.4 (R): now also G39.3
- net at G12.5 (Q): now also G40.1 (D)
- net AL0-7_OE: now reaches V6.3
- net at V5.1: now also U13.3
- net at V5.2: now also V46.3
- net at V110.3: now also V112.2
- net 59_RAMCS_OUT: now reaches V110.4
- net at H67.2: now also H51.3
- net 32_RIC12_A7_OUT: now reaches H67.3
- net 45_AL7_OUT: now reaches V1.1
- net 45_AL7_OUT: now also V33. (~{Q3})
- net at V1.3: now also V31.1
- net at D11.2: now also D3.5
- net at D11.3: now also C4.1 (D)
- net 54_AL3_OUT: now reaches U13.1
- net 54_AL3_OUT: now also T4. (~{Q3})
- net 47_AL6_OUT: now reaches V3.1
- net 47_AL6_OUT: now also V33. (~{Q3})
- net 54_AL3_IN: now reaches V46.1
- net 54_AL3_IN: now also V61. (~{Q3})
- net 51_AL4_OUT: now reaches U45.1
- net 51_AL4_OUT: now also V33. (~{Q3})
- net at U45.3: now also U47.1
- net 64_P34_IN: now reaches V33. (~{Q3})
- net 64_P34_IN: now also U31. (~{Q3}), V48. (~{Q3})
- net at G32.1: now also K34. (~{Q3})
- net at H51.1: now also K34. (~{Q3})
- net 49_AL5_IN: now reaches V77.1
- net at V77.3: now also U16.2
- net at A96.2: now also G33.3
- net 19_RIC12_A3_OUT: now reaches A96.3
- net 56_AL2_IN: now reaches V32.1
- net 56_AL2_IN: now also V61. (~{Q3})
- net 26_RIC12_A4_OUT: now reaches C69.3
- net 71_P30_IN: now reaches T4. (~{Q3})
- net 71_P30_IN: now also T17. (~{Q3}), T33. (~{Q3})
- net at G33.1: now also K34. (~{Q3})
- new net: P28.4, T4. (~{Q3}), V33. (~{Q3})
- new net 61_P37_IN: U31. (~{Q3}), V33. (~{Q3}), V48. (~{Q3})
- new net 62_P36_IN: U31. (~{Q3}), V33. (~{Q3}), V48. (~{Q3})
- new net 63_P35_IN: U31. (~{Q3}), V33. (~{Q3}), V48. (~{Q3})
- new net 65_P33_IN: T17. (~{Q3}), T33. (~{Q3}), T4. (~{Q3})
- new net 66_P32_IN: T17. (~{Q3}), T33. (~{Q3}), T4. (~{Q3})
- new net 67_P31_IN: T17. (~{Q3}), T33. (~{Q3}), T4. (~{Q3})
- new net 69_AS_IN: P28.1
- new net AD_LATCHED_4: K34. (~{Q3})
- new net AD_LATCHED_5: K34. (~{Q3})
- new net AD_LATCHED_6: K34. (~{Q3})
- new net AD_LATCHED_7: K34. (~{Q3})
Other:
- note added: "Either a schmidt trigger or a sync latch and I'm missing the clock input"
- note added: "TODO"
- note added: "unconnected?"
